File: PCB/LightsPCB/LightsPCB.kicad_pcb (KiCad board)
At the start: 2 copper layers, 56 x 56 mm, 13 parts

Commit message: Add files via upload
Parts:
- ?: renamed from Photosensor; footprint Resistors_ThroughHole:Resistor_Vertical_RM5mm -> Sensor:Resistor_Vertical_RM5mm
Routing:
- net GND: track 278.1 -> 260.4 mm, vias 5 -> 4
- net +5V: track 213.5 -> 213.0 mm
Other:
- board text added: "Aug 2016"
- board text added: "EN"
- board text added: "LIGHTS PCB V 1.0"
- board text added: "MCD"
- board text added: "RX"
- board text added: "STATE"
- board text added: "TX"
- board text added: "VCC"
